Commit message: fixed motion planning

File: config/so100_arm.ros2_control.xacro (robot description, xacro)
@@ -1,5 +1,5 @@
 <?xml version="1.0"?>
 <robot xmlns:xacro="http://www.ros.org/wiki/xacro">
-  <xacro:macro name="so100_bidirectional_ros2_control" params="name use_serial serial_port serial_baudrate calibration_file use_fake_hardware:=false">
+  <xacro:macro name="so100_arm_ros2_control" params="name use_serial serial_port serial_baudrate calibration_file use_fake_hardware:=false">
     <ros2_control name="${name}" type="system">
       <hardware>
@@ -8,6 +8,6 @@
         </xacro:if>
         <xacro:unless value="${use_fake_hardware}">
-          <plugin>so100_bidirectional/SO100BidirectionalInterface</plugin>
-          <param name="use_serial">${use_serial}</param>
+          <plugin>so100_arm/SO100ArmInterface</plugin>
+          <param name="use_serial">true</param>
           <param name="serial_port">${serial_port}</param>
           <param name="serial_baudrate">${serial_baudrate}</param>

File: config/so100_arm.urdf.xacro (robot description, xacro)
@@ -1,8 +1,8 @@
 <?xml version="1.0"?>
-<robot xmlns:xacro="http://www.ros.org/wiki/xacro" name="so100_bidirectional">
+<robot xmlns:xacro="http://www.ros.org/wiki/xacro" name="so100_arm">
   <!-- Parameters -->
   <xacro:arg name="serial_port" default="/dev/ttyACM0"/>
   <xacro:arg name="use_fake_hardware" default="false"/>
-  <xacro:include filename="$(find so100_bidirectional)/config/so100_bidirectional.ros2_control.xacro"/>
+  <xacro:include filename="$(find so100_arm)/config/so100_arm.ros2_control.xacro"/>
   <!-- Dummy world link to avoid KDL root link inertia warning -->
   <link name="world"/>
@@ -18,5 +18,5 @@
       <origin xyz="0 0 0" rpy="0 0 1.57079"/>
       <geometry>
-        <mesh filename="package://so100_bidirectional/meshes/Base.STL" scale="1.0 1.0 1.0"/>
+        <mesh filename="package://so100_arm/meshes/Base.STL" scale="1.0 1.0 1.0"/>
       </geometry>
       <material name="black">
@@ -27,5 +27,5 @@
       <origin xyz="0 0 0" rpy="0 0 0"/>
       <geometry>
-        <mesh filename="package://so100_bidirectional/meshes/Base.STL" scale="1.0 1.0 1.0"/>
+        <mesh filename="package://so100_arm/meshes/Base.STL" scale="1.0 1.0 1.0"/>
       </geometry>
     </collision>
@@ -47,5 +47,5 @@
       <origin xyz="0 0 0" rpy="1.57079 0 1.57079"/>
       <geometry>
-        <mesh filename="package://so100_bidirectional/meshes/Shoulder_Rotation_Pitch.STL" scale="1.0 1.0 1.0"/>
+        <mesh filename="package://so100_arm/meshes/Shoulder_Rotation_Pitch.STL" scale="1.0 1.0 1.0"/>
       </geometry>
       <material name="blue">
@@ -56,5 +56,5 @@
       <origin xyz="0 0 0" rpy="0 0 0"/>
       <geometry>
-        <mesh filename="package://so100_bidirectional/meshes/Shoulder_Rotation_Pitch.STL" scale="1.0 1.0 1.0"/>
+        <mesh filename="package://so100_arm/meshes/Shoulder_Rotation_Pitch.STL" scale="1.0 1.0 1.0"/>
       </geometry>
     </collision>
@@ -76,5 +76,5 @@
       <origin xyz="0 0 0" rpy="1.57079 0 1.57079"/>
       <geometry>
-        <mesh filename="package://so100_bidirectional/meshes/Upper_Arm.STL" scale="1.0 1.0 1.0"/>
+        <mesh filename="package://so100_arm/meshes/Upper_Arm.STL" scale="1.0 1.0 1.0"/>
       </geometry>
       <material name="green">
@@ -85,5 +85,5 @@
       <origin xyz="0 0 0" rpy="0 0 0"/>
       <geometry>
-        <mesh filename="package://so100_bidirectional/meshes/Upper_Arm.STL" scale="1.0 1.0 1.0"/>
+        <mesh filename="package://so100_arm/meshes/Upper_Arm.STL" scale="1.0 1.0 1.0"/>
       </geometry>
     </collision>
@@ -105,5 +105,5 @@
       <origin xyz="0 0 0" rpy="1.57079 0 1.57079"/>
       <geometry>
-        <mesh filename="package://so100_bidirectional/meshes/Lower_Arm.STL" scale="1.0 1.0 1.0"/>
+        <mesh filename="package://so100_arm/meshes/Lower_Arm.STL" scale="1.0 1.0 1.0"/>
       </geometry>
       <material name="red">
@@ -114,5 +114,5 @@
       <origin xyz="0 0 0" rpy="0 0 0"/>
       <geometry>
-        <mesh filename="package://so100_bidirectional/meshes/Lower_Arm.STL" scale="1.0 1.0 1.0"/>
+        <mesh filename="package://so100_arm/meshes/Lower_Arm.STL" scale="1.0 1.0 1.0"/>
       </geometry>
     </collision>
@@ -134,5 +134,5 @@
       <origin xyz="0 0 0" rpy="0 0 1.57079"/>
       <geometry>
-        <mesh filename="package://so100_bidirectional/meshes/Wrist_Pitch_Roll.STL" scale="1.0 1.0 1.0"/>
+        <mesh filename="package://so100_arm/meshes/Wrist_Pitch_Roll.STL" scale="1.0 1.0 1.0"/>
       </geometry>
       <material name="yellow">
@@ -143,5 +143,5 @@
       <origin xyz="0 0 0" rpy="0 0 0"/>
       <geometry>
-        <mesh filename="package://so100_bidirectional/meshes/Wrist_Pitch_Roll.STL" scale="1.0 1.0 1.0"/>
+        <mesh filename="package://so100_arm/meshes/Wrist_Pitch_Roll.STL" scale="1.0 1.0 1.0"/>
       </geometry>
     </collision>
@@ -163,5 +163,5 @@
       <origin xyz="0 0 0" rpy="0 0 0"/>
       <geometry>
-        <mesh filename="package://so100_bidirectional/meshes/Fixed_Gripper.STL" scale="1.0 1.0 1.0"/>
+        <mesh filename="package://so100_arm/meshes/Fixed_Gripper.STL" scale="1.0 1.0 1.0"/>
       </geometry>
       <material name="cyan">
@@ -172,5 +172,5 @@
       <origin xyz="0 0 0" rpy="0 0 0"/>
       <geometry>
-        <mesh filename="package://so100_bidirectional/meshes/Fixed_Gripper.STL" scale="1.0 1.0 1.0"/>
+        <mesh filename="package://so100_arm/meshes/Fixed_Gripper.STL" scale="1.0 1.0 1.0"/>
       </geometry>
     </collision>
@@ -192,5 +192,5 @@
       <origin xyz="0 0 0" rpy="0 0 0"/>
       <geometry>
-        <mesh filename="package://so100_bidirectional/meshes/Moving_Jaw.STL" scale="1.0 1.0 1.0"/>
+        <mesh filename="package://so100_arm/meshes/Moving_Jaw.STL" scale="1.0 1.0 1.0"/>
       </geometry>
       <material name="magenta">
@@ -201,5 +201,5 @@
       <origin xyz="0 0 0" rpy="0 0 0"/>
       <geometry>
-        <mesh filename="package://so100_bidirectional/meshes/Moving_Jaw.STL" scale="1.0 1.0 1.0"/>
+        <mesh filename="package://so100_arm/meshes/Moving_Jaw.STL" scale="1.0 1.0 1.0"/>
       </geometry>
     </collision>
@@ -217,10 +217,10 @@
   <link name="end_effector_link"/>
   <!-- ROS2 Control -->
-  <xacro:so100_bidirectional_ros2_control
-    name="SO100BidirectionalHardware"
+  <xacro:so100_arm_ros2_control
+    name="SO100ArmHardware"
     use_serial="true"
     serial_port="$(arg serial_port)"
     serial_baudrate="1000000"
     use_fake_hardware="$(arg use_fake_hardware)"
-    calibration_file="$(find so100_bidirectional)/config/calibration.yaml"/>
+    calibration_file="$(find so100_arm)/config/calibration.yaml"/>
 </robot>
